Commit message: adding colors and base link

File: description/robot_core.xacro (robot description, xacro)
@@ -1,4 +1,16 @@
 <?xml version="1.0"?>
-<robot xmlns:xacro="http://www.ros.org/wiki/xacro"  name="robot">
+<robot xmlns:xacro="http://www.ros.org/wiki/xacro">
     <xacro:include filename="robot_core.xacro" />
+    <material name="white">
+        <color rgba = "1 1 1 1"/>
+    </material>
+    <material name="orange">
+        <color rgba = "1 0.3 0.1 1"/>
+    </material>
+    <material name="blue">
+        <color rgba = "0.2 0.2 1 1"/>
+    </material>
+    <material name="black">
+        <color rgba = "0 0 0 1"/>
+    </material>
 </robot>

Commit message: adding colors and base link

File: description/robot_core.xacro (robot description, xacro)
@@ -14,3 +14,5 @@
         <color rgba = "0 0 0 1"/>
     </material>
+    <link name="base_link">
+    </link>
 </robot>

Commit message: commit changes

File: description/robot_core.xacro (robot description, xacro)
@@ -16,3 +16,17 @@
     <link name="base_link">
     </link>
+    <joint name="chassis_joint" type="fixed">
+    <parent link="base_link"/>
+    <child link="chassis"/>
+    <origin xyz="-0.1 0 0"/>
+    </joint>
+    <link name="chassis">
+    <visual>
+        <origin xyz="0.15 0 0.075" rpy="0 0 0"/>
+        <geometry>
+            <box size="0.3 0.3 0.15"/>
+        </geometry>
+        <material name="white"/>
+    </visual>
+    </link>
 </robot>

Commit message: updated robot_core.xacro

File: description/robot_core.xacro (robot description, xacro)
@@ -1,5 +1,4 @@
 <?xml version="1.0"?>
-<robot xmlns:xacro="http://www.ros.org/wiki/xacro">
-    <xacro:include filename="robot_core.xacro" />
+<robot xmlns:xacro="http://www.ros.org/wiki/xacro" >
     <material name="white">
         <color rgba = "1 1 1 1"/>
@@ -30,3 +29,47 @@
     </visual>
     </link>
+    <!-- L Wheel -->
+    <joint name="left_wheel_joint" type="continuous">
+        <parent link="base_link"/>
+        <child link="left_wheel"/>
+        <origin xyz="0 0.175 0" rpy="-${pi/2} 0 0"/>
+        <axis xyz="0 0 1"/>
+    </joint>
+    <link name="left_wheel">
+        <visual>
+            <geometry>
+                <cylinder length="0.04" radius="0.05" />
+            </geometry>
+            <material name="black"/>
+        </visual>
+    </link>
+    <!-- R Wheel -->
+    <joint name="right_wheel_joint" type="continuous">
+        <parent link="base_link"/>
+        <child link="right_wheel"/>
+        <origin xyz="0 -0.175 0" rpy="${pi/2} 0 0"/>
+        <axis xyz="0 0 -1"/>
+    </joint>
+    <link name="right_wheel">
+        <visual>
+            <geometry>
+                <cylinder length="0.04" radius="0.05" />
+            </geometry>
+            <material name="black"/>
+        </visual>
+    </link>
+    <!-- Caster Wheel -->
+    <joint name="caster_wheel_joint" type="fixed">
+        <parent link="chassis"/>
+        <child link="caster_wheel"/>
+        <origin xyz="0.24 0 0" rpy="0 0 0"/>
+    </joint>
+    <link name="caster_wheel">
+        <visual>
+            <geometry>
+                <sphere radius="0.05" />
+            </geometry>
+            <material name="blue"/>
+        </visual>
+    </link>
 </robot>

Commit message: no message

File: description/robot_core.xacro (robot description, xacro)
@@ -24,5 +24,5 @@
         <origin xyz="0.15 0 0.075" rpy="0 0 0"/>
         <geometry>
-            <box size="0.3 0.3 0.15"/>
+            <box size="0.3 0.3 0.10"/>
         </geometry>
         <material name="white"/>
